Commit message: Add support for multirobot simulation/rviz

File: turtlebot3_description/urdf/turtlebot3_burger.rviz.urdf.xacro (robot description, xacro)
@@ -3,13 +3,14 @@
   <xacro:include filename="$(find turtlebot3_description)/urdf/common_properties.xacro"/>
   <xacro:include filename="$(find turtlebot3_description)/urdf/turtlebot3_burger.gazebo.xacro"/>
+  <xacro:arg name="prefix" default=""/>
   <xacro:arg name="robot_color" default=""/>
   <xacro:property name="color" value="$(arg robot_color)"/>
-  <link name="base_footprint"/>
-  <joint name="base_joint" type="fixed">
-    <parent link="base_footprint"/>
-    <child link="base_link"/>
+  <link name="$(arg prefix)/base_footprint"/>
+  <joint name="$(arg prefix)/base_joint" type="fixed">
+    <parent link="$(arg prefix)/base_footprint"/>
+    <child link="$(arg prefix)/base_link"/>
     <origin xyz="0.0 0.0 0.010" rpy="0 0 0"/>
   </joint>
-  <link name="base_link">
+  <link name="$(arg prefix)/base_link">
     <visual>
       <origin xyz="-0.032 0 0.0" rpy="0 0 0"/>
@@ -33,11 +34,11 @@
     </inertial>
   </link>
-  <joint name="wheel_left_joint" type="continuous">
-    <parent link="base_link"/>
-    <child link="wheel_left_link"/>
+  <joint name="$(arg prefix)/wheel_left_joint" type="continuous">
+    <parent link="$(arg prefix)/base_link"/>
+    <child link="$(arg prefix)/wheel_left_link"/>
     <origin xyz="0.0 0.08 0.023" rpy="-1.57 0 0"/>
     <axis xyz="0 0 1"/>
   </joint>
-  <link name="wheel_left_link">
+  <link name="$(arg prefix)/wheel_left_link">
     <visual>
       <origin xyz="0 0 0" rpy="1.57 0 0"/>
@@ -61,11 +62,11 @@
       </inertial>
   </link>
-  <joint name="wheel_right_joint" type="continuous">
-    <parent link="base_link"/>
-    <child link="wheel_right_link"/>
+  <joint name="$(arg prefix)/wheel_right_joint" type="continuous">
+    <parent link="$(arg prefix)/base_link"/>
+    <child link="$(arg prefix)/wheel_right_link"/>
     <origin xyz="0.0 -0.080 0.023" rpy="-1.57 0 0"/>
     <axis xyz="0 0 1"/>
   </joint>
-  <link name="wheel_right_link">
+  <link name="$(arg prefix)/wheel_right_link">
     <visual>
       <origin xyz="0 0 0" rpy="1.57 0 0"/>
@@ -89,10 +90,10 @@
       </inertial>
   </link>
-  <joint name="caster_back_joint" type="fixed">
-    <parent link="base_link"/>
-    <child link="caster_back_link"/>
+  <joint name="$(arg prefix)/caster_back_joint" type="fixed">
+    <parent link="$(arg prefix)/base_link"/>
+    <child link="$(arg prefix)/caster_back_link"/>
     <origin xyz="-0.081 0 -0.004" rpy="-1.57 0 0"/>
   </joint>
-  <link name="caster_back_link">
+  <link name="$(arg prefix)/caster_back_link">
     <collision>
       <origin xyz="0 0.001 0" rpy="0 0 0"/>
@@ -109,16 +110,16 @@
     </inertial>
   </link>
-  <joint name="imu_joint" type="fixed">
-    <parent link="base_link"/>
-    <child link="imu_link"/>
+  <joint name="$(arg prefix)/imu_joint" type="fixed">
+    <parent link="$(arg prefix)/base_link"/>
+    <child link="$(arg prefix)/imu_link"/>
     <origin xyz="-0.032 0 0.068" rpy="0 0 0"/>
   </joint>
-  <link name="imu_link"/>
-  <joint name="scan_joint" type="fixed">
-    <parent link="base_link"/>
-    <child link="base_scan"/>
+  <link name="$(arg prefix)/imu_link"/>
+  <joint name="$(arg prefix)/scan_joint" type="fixed">
+    <parent link="$(arg prefix)/base_link"/>
+    <child link="$(arg prefix)/base_scan"/>
     <origin xyz="-0.032 0 0.172" rpy="0 0 0"/>
   </joint>
-  <link name="base_scan">
+  <link name="$(arg prefix)/base_scan">
     <visual>
       <origin xyz="0 0 0.0" rpy="0 0 0"/>
